Commit message: Some additions to debug sensor simulation

File: urdf/standardrobots_oasis300.xacro (robot description, xacro)
@@ -56,6 +56,6 @@
         <parent link="${base_link}"/>
         <child link="livox_base"/>
-        <origin rpy="0 0 1.5707"
-                xyz="0.0 0.4 0.3057"/>
+        <origin rpy="0 0.0 1.5707"
+                xyz="0.0 0.7 0.3057"/>
     </joint>
     </xacro:macro>
