Commit message: Add gpu support to livox mid 360 lidar

File: urdf/livox_mid360.xacro (robot description, xacro)
@@ -3,10 +3,9 @@
   <xacro:property name="M_PI" value="3.14159"/>
   <xacro:property name="laser_min_range" value="0.1"/>
-  <xacro:property name="laser_max_range" value="40.0"/>
-  <xacro:property name="horizontal_fov" value="180.0"/>
-  <xacro:property name="vertical_fov_max" value="52.0"/>
-  <xacro:property name="vertical_fov_min" value="-7.0"/>
+  <xacro:property name="laser_max_range" value="200.0"/>
+  <xacro:property name="horizontal_fov" value="70.4"/>
+  <xacro:property name="vertical_fov" value="70.4"/>
   <xacro:property name="ros_topic" value="scan"/>
-  <xacro:property name="samples" value="20000"/>
+  <xacro:property name="samples" value="10000"/>
   <xacro:property name="downsample" value="1"/>
   <xacro:macro name="null_inertial">
@@ -18,43 +17,69 @@
     </inertial>
   </xacro:macro>
-  <xacro:macro name="Livox_Mid_gazebo_sensor" params="link:=blabla visualize:=True update_rate:=10 resolution:=0.02 noise_mean:=0.0 noise_stddev:=0.01 name:=livox ros_topic:=scan">
-    <gazebo reference="front_mount_link">
+  <xacro:macro name="Livox_Mid_gazebo_sensor" params="visualize:=True update_rate:=10 resolution:=0.002 noise_mean:=0.0 noise_stddev:=0.0 name:=livox">
+    <gazebo reference="${name}">
       <sensor type="ray" name="laser_${name}">
         <pose>0 0 0 0 0 0</pose>
         <visualize>${visualize}</visualize>
         <update_rate>${update_rate}</update_rate>
+        <ray>
+          <scan>
+            <horizontal>
+              <samples>100</samples>
+              <resolution>1</resolution>
+              <min_angle>${-horizontal_fov/360*M_PI}</min_angle>
+              <max_angle>${horizontal_fov/360*M_PI}</max_angle>
+            </horizontal>
+            <vertical>
+              <samples>50</samples>
+              <resolution>1</resolution>
+              <min_angle>${-vertical_fov/360*M_PI}</min_angle>
+              <max_angle>${vertical_fov/360*M_PI}</max_angle>
+            </vertical>
+          </scan>
+          <range>
+            <min>${laser_min_range}</min>
+            <max>${laser_max_range}</max>
+            <resolution>${resolution}</resolution>
+          </range>
+          <noise>
+            <type>gaussian</type>
+            <mean>${noise_mean}</mean>
+            <stddev>${noise_stddev}</stddev>
+          </noise>
+        </ray>
         <!-- This ray plgin is only for visualization. -->
         <plugin name="gazebo_ros_laser_controller" filename="liblivox_laser_simulation.so">
-			<ray>
-			  <scan>
-				<horizontal>
-				<samples>100</samples>
-				<resolution>1</resolution>
-				<min_angle>${-horizontal_fov/180*M_PI}</min_angle>
-				<max_angle>${horizontal_fov/180*M_PI}</max_angle>
-				</horizontal>
-				<vertical>
-				<samples>50</samples>
-				<resolution>1</resolution>
-				<min_angle>${vertical_fov_min/180*M_PI}</min_angle>
-				<max_angle>${vertical_fov_max/180*M_PI}</max_angle>
-				</vertical>
-			  </scan>
-			  <range>
-				<min>${laser_min_range}</min>
-				<max>${laser_max_range}</max>
-				<resolution>${resolution}</resolution>
-			  </range>
-			  <noise>
-				<type>gaussian</type>
-				<mean>${noise_mean}</mean>
-				<stddev>${noise_stddev}</stddev>
-			  </noise>
-			</ray>
+          <ray>
+            <scan>
+              <horizontal>
+                <samples>100</samples>
+                <resolution>1</resolution>
+                <min_angle>${-horizontal_fov/360*M_PI}</min_angle>
+                <max_angle>${horizontal_fov/360*M_PI}</max_angle>
+              </horizontal>
+              <vertical>
+                <samples>50</samples>
+                <resolution>1</resolution>
+                <min_angle>${-vertical_fov/360*M_PI}</min_angle>
+                <max_angle>${vertical_fov/360*M_PI}</max_angle>
+              </vertical>
+            </scan>
+            <range>
+              <min>${laser_min_range}</min>
+              <max>${laser_max_range}</max>
+              <resolution>${resolution}</resolution>
+            </range>
+            <noise>
+              <type>gaussian</type>
+              <mean>${noise_mean}</mean>
+              <stddev>${noise_stddev}</stddev>
+            </noise>
+          </ray>
           <visualize>${visualize}</visualize>
-		  <samples>${samples}</samples>
-		  <downsample>${downsample}</downsample>
-		  <csv_file_name>package://livox_laser_simulation/scan_mode/mid360.csv</csv_file_name>
-		  <ros_topic>${ros_topic}</ros_topic>
+          <samples>${samples}</samples>
+          <downsample>${downsample}</downsample>
+          <csv_file_name>package://livox_laser_simulation/scan_mode/mid360.csv</csv_file_name>
+          <ros_topic>${ros_topic}</ros_topic>
         </plugin>
       </sensor>
@@ -65,18 +90,17 @@
       <xacro:null_inertial/>
       <visual>
-        <origin xyz="0 0 0" rpy="0 0 0"/>
+        <origin xyz="0.00 0 0.00" rpy="0 0 0"/>
         <geometry>
-          <mesh filename="package://livox_laser_simulation/meshes/livox_mid360.stl">
+          <mesh filename="package://livox_laser_simulation/meshes/livox_mid40.dae">
           </mesh>
         </geometry>
       </visual>
-      <!--
       <collision>
-          <origin xyz="0 0 -0.047" rpy="0 0 0" />
+          <origin xyz="0 0 0" rpy="0 0 0" />
           <geometry>
-          <mesh filename="package://livox_laser_simulation/meshes/livox_mid360.stl">
+          <mesh filename="package://livox_laser_simulation/meshes/livox_mid40.dae">
           </mesh>
           </geometry>
-      </collision>-->
+      </collision>
     </link>
     <link name="${name}">
@@ -86,9 +110,9 @@
       <parent link="${name}_base"/>
       <child link="${name}"/>
-      <origin rpy="0 0 0" xyz="0.0 0.0 0.047"/>
+      <origin rpy="0 0 0" xyz="0.0 0.0 0.0"/>
     </joint>
     <xacro:Livox_Mid_gazebo_sensor name="${name}" visualize="${visualize}"/>
   </xacro:macro>
-  <xacro:Livox_Mid360 name="livox"/>
+    <xacro:Livox_Mid360 name="livox"/>
   <xacro:include filename="$(find livox_laser_simulation)/urdf/standardrobots_oasis300.xacro"/>
   <xacro:link_oasis name="oasis"/>

Commit message: Fix cpu based simulation and add gpu based into xacro file

File: urdf/livox_mid360.xacro (robot description, xacro)
@@ -4,27 +4,22 @@
   <xacro:property name="laser_min_range" value="0.1"/>
   <xacro:property name="laser_max_range" value="200.0"/>
-  <xacro:property name="horizontal_fov" value="70.4"/>
-  <xacro:property name="vertical_fov" value="70.4"/>
+  <xacro:property name="horizontal_fov" value="360"/>
+  <xacro:property name="vertical_fov_min" value="-180.0"/>
+  <xacro:property name="vertical_fov_max" value="180.0"/>
   <xacro:property name="ros_topic" value="scan"/>
-  <xacro:property name="samples" value="10000"/>
+  <xacro:property name="samples" value="20000"/>
   <xacro:property name="downsample" value="1"/>
-  <xacro:macro name="null_inertial">
-    <inertial>
-      <mass value="0.1"/>
-    <inertia ixx="0.01" ixy="0" ixz="0"
-          iyy="0.01" iyz="0"
-          izz="0.01"/>
-    </inertial>
-  </xacro:macro>
-  <xacro:macro name="Livox_Mid_gazebo_sensor" params="visualize:=True update_rate:=10 resolution:=0.002 noise_mean:=0.0 noise_stddev:=0.0 name:=livox">
+  <xacro:property name="gpu_enabled" value="true"/>
+  <!-- CPU Simulation -->
+  <xacro:macro name="livox_mid_gazebo_sensor" params="visualize:=False update_rate:=10 resolution:=0.002 noise_mean:=0.0 noise_stddev:=0.0 name:=livox ros_topic:=/scan">
     <gazebo reference="${name}">
-      <sensor type="ray" name="laser_${name}">
+      <sensor type="ray" name="${name}">
         <pose>0 0 0 0 0 0</pose>
-        <visualize>${visualize}</visualize>
+        <visualize>false</visualize>
         <update_rate>${update_rate}</update_rate>
         <ray>
           <scan>
             <horizontal>
-              <samples>100</samples>
+              <samples>1</samples>
               <resolution>1</resolution>
               <min_angle>${-horizontal_fov/360*M_PI}</min_angle>
@@ -32,8 +27,8 @@
             </horizontal>
             <vertical>
-              <samples>50</samples>
+              <samples>1</samples>
               <resolution>1</resolution>
-              <min_angle>${-vertical_fov/360*M_PI}</min_angle>
-              <max_angle>${vertical_fov/360*M_PI}</max_angle>
+              <min_angle>${vertical_fov_min/180*M_PI}</min_angle>
+              <max_angle>${vertical_fov_max/180*M_PI}</max_angle>
             </vertical>
           </scan>
@@ -54,5 +49,5 @@
             <scan>
               <horizontal>
-                <samples>100</samples>
+                <samples>200</samples>
                 <resolution>1</resolution>
                 <min_angle>${-horizontal_fov/360*M_PI}</min_angle>
@@ -60,8 +55,8 @@
               </horizontal>
               <vertical>
-                <samples>50</samples>
+                <samples>100</samples>
                 <resolution>1</resolution>
-                <min_angle>${-vertical_fov/360*M_PI}</min_angle>
-                <max_angle>${vertical_fov/360*M_PI}</max_angle>
+                <min_angle>${vertical_fov_min/180*M_PI}</min_angle>
+                <max_angle>${vertical_fov_max/180*M_PI}</max_angle>
               </vertical>
             </scan>
@@ -86,34 +81,110 @@
     </gazebo>
   </xacro:macro>
-  <xacro:macro name="Livox_Mid360" params="visualize:=True name:=livox">
+  <!-- GPU Simulation -->
+  <xacro:macro name="livox_mid_gazebo_gpu_sensor" params="visualize:=False update_rate:=10 samples:=20000 resolution:=0.002 noise_mean:=0.0 noise_stddev:=0.0 name:=livox ros_topic:=/scan">
+    <gazebo reference="${name}">
+      <sensor type="gpu_ray" name="${name}">
+        <pose>0 0 0 0 0 0</pose>
+        <visualize>${visualize}</visualize>
+        <update_rate>${update_rate}</update_rate>
+        <sample_sensor>True</sample_sensor>
+        <sample_size>${samples}</sample_size>
+        <sample_csv_file>package://livox_laser_simulation/scan_mode/mid360.csv</sample_csv_file>
+        <ray>
+          <scan>
+            <horizontal>
+              <samples>1</samples>
+              <resolution>1</resolution>
+              <min_angle>${-horizontal_fov/360*M_PI}</min_angle>
+              <max_angle>${horizontal_fov/360*M_PI}</max_angle>
+            </horizontal>
+            <vertical>
+              <samples>1</samples>
+              <resolution>1</resolution>
+              <min_angle>${vertical_fov_min/180*M_PI}</min_angle>
+              <max_angle>${vertical_fov_max/180*M_PI}</max_angle>
+            </vertical>
+          </scan>
+          <range>
+            <min>${laser_min_range}</min>
+            <max>${laser_max_range}</max>
+            <resolution>${resolution}</resolution>
+          </range>
+          <noise>
+            <type>gaussian</type>
+            <mean>${noise_mean}</mean>
+            <stddev>${noise_stddev}</stddev>
+          </noise>
+        </ray>
+        <!-- This ray plgin is only for visualization. -->
+        <plugin name="gazebo_ros_gpu_laser_controller" filename="liblivox_laser_gpu_simulation.so">
+          <ray>
+            <scan>
+              <horizontal>
+                <samples>1</samples>
+                <resolution>1</resolution>
+                <min_angle>${-horizontal_fov/360*M_PI}</min_angle>
+                <max_angle>${horizontal_fov/360*M_PI}</max_angle>
+              </horizontal>
+              <vertical>
+                <samples>1</samples>
+                <resolution>1</resolution>
+                <min_angle>${vertical_fov_min/180*M_PI}</min_angle>
+                <max_angle>${vertical_fov_max/180*M_PI}</max_angle>
+              </vertical>
+            </scan>
+            <range>
+              <min>${laser_min_range}</min>
+              <max>${laser_max_range}</max>
+              <resolution>${resolution}</resolution>
+            </range>
+            <noise>
+              <type>gaussian</type>
+              <mean>${noise_mean}</mean>
+              <stddev>${noise_stddev}</stddev>
+            </noise>
+          </ray>
+          <visualize>${visualize}</visualize>
+          <samples>${samples}</samples>
+          <downsample>${downsample}</downsample>
+          <csv_file_name>package://livox_laser_simulation/scan_mode/mid360.csv</csv_file_name>
+          <ros_topic>${ros_topic}</ros_topic>
+        </plugin>
+      </sensor>
+    </gazebo>
+  </xacro:macro>
+  <xacro:macro name="livox_mid360" params="visualize:=False name:=livox parent:=livox_base ros_topic:=/scan gpu_enabled:=False">
+    <!-- base -->
+    <joint name="${name}_joint" type="fixed">
+      <origin rpy="0 0 0" xyz="0.0 0.0 0.0"/>
+      <parent link="${parent}"/>
+      <child link="${name}_base"/>
+    </joint>
     <link name="${name}_base">
-      <xacro:null_inertial/>
       <visual>
-        <origin xyz="0.00 0 0.00" rpy="0 0 0"/>
+        <origin xyz="0 0 0" rpy="0 0 0"/>
         <geometry>
-          <mesh filename="package://livox_laser_simulation/meshes/livox_mid40.dae">
+          <mesh filename="package://common_description/meshes/livox/livox_mid_360.stl">
           </mesh>
         </geometry>
       </visual>
-      <collision>
-          <origin xyz="0 0 0" rpy="0 0 0" />
-          <geometry>
-          <mesh filename="package://livox_laser_simulation/meshes/livox_mid40.dae">
-          </mesh>
-          </geometry>
-      </collision>
     </link>
-    <link name="${name}">
-      <xacro:null_inertial/>
-    </link>
-    <joint name="${name}_to_${name}_base_joint" type="fixed">
+    <joint name="${name}_base_mount_joint" type="fixed">
+      <origin rpy="0 0 0" xyz="0.0 0.0 0.047"/>
       <parent link="${name}_base"/>
       <child link="${name}"/>
-      <origin rpy="0 0 0" xyz="0.0 0.0 0.0"/>
     </joint>
-    <xacro:Livox_Mid_gazebo_sensor name="${name}" visualize="${visualize}"/>
+    <link name="${name}"/>
+    <xacro:if value="${gpu_enabled}">
+      <!-- GPU based simulation -->
+      <xacro:livox_mid_gazebo_gpu_sensor name="${name}" visualize="${visualize}" ros_topic="${ros_topic}"/>
+    </xacro:if>
+    <xacro:unless value="${gpu_enabled}">
+      <!-- CPU based simulation -->
+      <xacro:livox_mid_gazebo_sensor name="${name}" visualize="True" ros_topic="${ros_topic}"/>
+    </xacro:unless>
   </xacro:macro>
-    <xacro:Livox_Mid360 name="livox"/>
+  <!--<xacro:livox_mid360 name="livox"/>
   <xacro:include filename="$(find livox_laser_simulation)/urdf/standardrobots_oasis300.xacro"/>
-  <xacro:link_oasis name="oasis"/>
+  <xacro:link_oasis name="oasis"/>-->
 </robot>

File: urdf/livox_mid360_gpu.xacro (robot description, xacro)
@@ -10,15 +10,79 @@
   <xacro:property name="samples" value="20000"/>
   <xacro:property name="downsample" value="1"/>
-  <xacro:macro name="null_inertial">
-    <inertial>
-      <mass value="0.1"/>
-    <inertia ixx="0.01" ixy="0" ixz="0"
-          iyy="0.01" iyz="0"
-          izz="0.01"/>
-    </inertial>
+  <xacro:property name="gpu_enabled" value="true"/>
+  <!-- CPU Simulation -->
+  <xacro:macro name="livox_mid_gazebo_sensor" params="visualize:=False update_rate:=10 resolution:=0.002 noise_mean:=0.0 noise_stddev:=0.0 name:=livox ros_topic:=/scan">
+    <gazebo reference="${name}">
+      <sensor type="ray" name="${name}">
+        <pose>0 0 0 0 0 0</pose>
+        <visualize>${visualize}</visualize>
+        <update_rate>${update_rate}</update_rate>
+        <ray>
+          <scan>
+            <horizontal>
+              <samples>1</samples>
+              <resolution>1</resolution>
+              <min_angle>${-horizontal_fov/360*M_PI}</min_angle>
+              <max_angle>${horizontal_fov/360*M_PI}</max_angle>
+            </horizontal>
+            <vertical>
+              <samples>1</samples>
+              <resolution>1</resolution>
+              <min_angle>${vertical_fov_min/180*M_PI}</min_angle>
+              <max_angle>${vertical_fov_max/180*M_PI}</max_angle>
+            </vertical>
+          </scan>
+          <range>
+            <min>${laser_min_range}</min>
+            <max>${laser_max_range}</max>
+            <resolution>${resolution}</resolution>
+          </range>
+          <noise>
+            <type>gaussian</type>
+            <mean>${noise_mean}</mean>
+            <stddev>${noise_stddev}</stddev>
+          </noise>
+        </ray>
+        <!-- This ray plgin is only for visualization. -->
+        <plugin name="gazebo_ros_laser_controller" filename="liblivox_laser_simulation.so">
+          <ray>
+            <scan>
+              <horizontal>
+                <samples>200</samples>
+                <resolution>1</resolution>
+                <min_angle>${-horizontal_fov/360*M_PI}</min_angle>
+                <max_angle>${horizontal_fov/360*M_PI}</max_angle>
+              </horizontal>
+              <vertical>
+                <samples>100</samples>
+                <resolution>1</resolution>
+                <min_angle>${vertical_fov_min/180*M_PI}</min_angle>
+                <max_angle>${vertical_fov_max/180*M_PI}</max_angle>
+              </vertical>
+            </scan>
+            <range>
+              <min>${laser_min_range}</min>
+              <max>${laser_max_range}</max>
+              <resolution>${resolution}</resolution>
+            </range>
+            <noise>
+              <type>gaussian</type>
+              <mean>${noise_mean}</mean>
+              <stddev>${noise_stddev}</stddev>
+            </noise>
+          </ray>
+          <visualize>${visualize}</visualize>
+          <samples>${samples}</samples>
+          <downsample>${downsample}</downsample>
+          <csv_file_name>package://livox_laser_simulation/scan_mode/mid360.csv</csv_file_name>
+          <ros_topic>${ros_topic}</ros_topic>
+        </plugin>
+      </sensor>
+    </gazebo>
   </xacro:macro>
-  <xacro:macro name="Livox_Mid_gazebo_sensor" params="visualize:=False update_rate:=10 samples:=20000 resolution:=0.002 noise_mean:=0.0 noise_stddev:=0.0 name:=livox ros_topic:=/scan">
+  <!-- GPU Simulation -->
+  <xacro:macro name="livox_mid_gazebo_gpu_sensor" params="visualize:=False update_rate:=10 samples:=20000 resolution:=0.002 noise_mean:=0.0 noise_stddev:=0.0 name:=livox ros_topic:=/scan">
     <gazebo reference="${name}">
-      <sensor type="gpu_ray" name="laser_${name}">
+      <sensor type="gpu_ray" name="${name}">
         <pose>0 0 0 0 0 0</pose>
         <visualize>${visualize}</visualize>
@@ -90,5 +154,5 @@
     </gazebo>
   </xacro:macro>
-  <xacro:macro name="Livox_Mid360" params="visualize:=False name:=livox parent:=livox_base ros_topic:=/scan">
+  <xacro:macro name="livox_mid360" params="visualize:=False name:=livox parent:=livox_base ros_topic:=/scan gpu_enabled:=False">
     <!-- base -->
     <joint name="${name}_joint" type="fixed">
@@ -98,9 +162,8 @@
     </joint>
     <link name="${name}_base">
-      <!--<xacro:null_inertial/>-->
       <visual>
         <origin xyz="0 0 0" rpy="0 0 0"/>
         <geometry>
-          <mesh filename="package://common_description/meshes/livox/livox_mid_360.stl">
+          <mesh filename="package://livox_laser_simulation/meshes/livox/livox_mid360.stl">
           </mesh>
         </geometry>
@@ -108,29 +171,19 @@
     </link>
     <joint name="${name}_base_mount_joint" type="fixed">
-      <origin rpy="0 0 0" xyz="0.0 0.0 0.0"/>
+      <origin rpy="0 0 0" xyz="0.0 0.0 0.047"/>
       <parent link="${name}_base"/>
       <child link="${name}"/>
     </joint>
     <link name="${name}"/>
-    <joint name="${name}_base_mount_joint2" type="fixed">
-      <origin rpy="0 0 0" xyz="0.0 0.0 0.0"/>
-      <parent link="${name}"/>
-      <child link="laser_${name}"/>
-    </joint>
-    <link name="laser_${name}"/>
-    <xacro:Livox_Mid_gazebo_sensor name="${name}" visualize="${visualize}" ros_topic="${ros_topic}"/>
-    <!--
-    <link name="${name}">
-      <xacro:null_inertial/>
-    </link>
-    -->
-    <!--<joint name="${name}_to_${name}_base_joint" type="fixed">
-      <parent link="${name}_base"/>
-      <child link="${name}"/>
-      <origin rpy="0 0 0" xyz="0.0 0.0 0.0"/>
-    </joint>-->
-    <!--<xacro:Livox_Mid_gazebo_sensor name="${name}" visualize="${visualize}"/>-->
+    <xacro:if value="${gpu_enabled}">
+      <!-- GPU based simulation -->
+      <xacro:livox_mid_gazebo_gpu_sensor name="${name}" visualize="${visualize}" ros_topic="${ros_topic}"/>
+    </xacro:if>
+    <xacro:unless value="${gpu_enabled}">
+      <!-- CPU based simulation -->
+      <xacro:livox_mid_gazebo_sensor name="${name}" visualize="${visualize}" ros_topic="${ros_topic}"/>
+    </xacro:unless>
   </xacro:macro>
-  <!--<xacro:Livox_Mid360 name="livox"/>
+  <!--<xacro:livox_mid360 name="livox"/>
   <xacro:include filename="$(find livox_laser_simulation)/urdf/standardrobots_oasis300.xacro"/>
   <xacro:link_oasis name="oasis"/>-->

File: urdf/standardrobots_oasis300.xacro (robot description, xacro)
@@ -56,6 +56,6 @@
         <parent link="${base_link}"/>
         <child link="livox_base"/>
-        <origin rpy="0 0.0 1.5707"
-                xyz="0.0 0.7 0.3057"/>
+        <origin rpy="0 0 ${M_PI/2}"
+                xyz="0.0 0.4 0.3057"/>
     </joint>
     </xacro:macro>
